Commit message: refactor: assemble steering into platform_description

File: src/platform_description/urdf/platform_base.xacro (robot description, xacro)
@@ -1,40 +1,4 @@
 <?xml version="1.0"?>
-<robot name="bolid" xmlns:xacro="http://www.ros.org/wiki/xacro">
-  <xacro:property name="wheel_radius" value="0.035"/>
-  <xacro:property name="wheel_width" value="0.010"/>
-  <xacro:property name="chassis_length" value="0.375"/>
-  <xacro:property name="chassis_width" value="0.125"/>
-  <xacro:property name="chassis_height" value="0.03"/>
-  <xacro:property name="max_steering_angle" value="0.6108" />
-  <xacro:property name="max_steering_angular_velocity" value="20.0" />
-  <xacro:property name="max_steering_effort" value="200.0" />
-  <xacro:property name="max_wheel_angular_velocity" value="100.0"/>
-  <xacro:property name="max_effort" value="30.0" />
-  <xacro:macro name="box_inertia" params="m l w h xyz rpy">
-      <inertial>
-          <origin xyz="${xyz}" rpy="${rpy}"/>
-          <mass value="${m}"/>
-          <inertia ixx="${(1/12) * m * (w*w + h*h)}" ixy="0.0" ixz="0.0"
-                   iyy="${(1/12) * m * (l*l + h*h)}" iyz="0.0"
-                   izz="${(1/12) * m * (l*l + w*w)}"/>
-      </inertial>
-  </xacro:macro>
-  <xacro:macro name="cylinder_inertia" params="m r h xyz rpy">
-      <inertial>
-          <origin xyz="${xyz}" rpy="${rpy}"/>
-          <mass value="${m}"/>
-          <inertia ixx="${(1/12) * m * (3*r*r + h*h)}" ixy="0.0" ixz="0.0"
-                   iyy="${(1/12) * m * (3*r*r + h*h)}" iyz="0.0"
-                   izz="${(1/2) * m * r*r}"/>
-      </inertial>
-  </xacro:macro>
-  <xacro:macro name="steering_inertia" params="">
-      <inertial>
-        <mass value="0.1"/>
-        <inertia ixx="1e-3" ixy="0.0" ixz="0.0" iyy="1e-3" iyz="0.0" izz="1e-3"/>
-      </inertial>
-  </xacro:macro>
-  <material name="red"> <color rgba="1 0 0 1"/> </material>
-  <material name="black"> <color rgba="0 0 0 1"/> </material>
+<robot xmlns:xacro="http://www.ros.org/wiki/xacro">
   <link name="base_footprint"/>
   <link name="base_link">
@@ -167,58 +131,3 @@
   <gazebo reference="base_link"><material>Gazebo/Red</material></gazebo>
   <gazebo reference="platform_link"><material>Gazebo/Red</material></gazebo>
-  <ros2_control name="control" type="system">
-    <hardware>
-      <plugin>gz_ros2_control/GazeboSimSystem</plugin>
-    </hardware>
-    <joint name="front_left_steering_joint">
-      <command_interface name="position">
-        <param name="min">${-max_steering_angle}</param>
-        <param name="max">${max_steering_angle}</param>
-      </command_interface>
-      <state_interface name="position"/>
-      <state_interface name="velocity"/>
-      <state_interface name="effort"/>
-    </joint>
-    <joint name="front_right_steering_joint">
-      <command_interface name="position">
-        <param name="min">${-max_steering_angle}</param>
-        <param name="max">${max_steering_angle}</param>
-      </command_interface>
-      <state_interface name="position"/>
-      <state_interface name="velocity"/>
-      <state_interface name="effort"/>
-    </joint>
-    <joint name="rear_left_wheel_joint">
-      <command_interface name="velocity">
-        <param name="min">${-max_wheel_angular_velocity}</param>
-        <param name="max">${max_wheel_angular_velocity}</param>
-      </command_interface>
-      <state_interface name="position"/>
-      <state_interface name="velocity"/>
-      <state_interface name="effort"/>
-    </joint>
-    <joint name="rear_right_wheel_joint">
-      <command_interface name="velocity">
-        <param name="min">${-max_wheel_angular_velocity}</param>
-        <param name="max">${max_wheel_angular_velocity}</param>
-      </command_interface>
-      <state_interface name="position"/>
-      <state_interface name="velocity"/>
-      <state_interface name="effort"/>
-    </joint>
-  </ros2_control>
-  <gazebo>
-    <plugin filename="gz-sim-joint-state-publisher-system" name="gz::sim::systems::JointStatePublisher">
-      <topic>joint_states</topic>
-      <joint_name>front_left_steering_joint</joint_name>
-      <joint_name>front_right_steering_joint</joint_name>
-      <joint_name>front_left_wheel_joint</joint_name>
-      <joint_name>front_right_wheel_joint</joint_name>
-      <joint_name>rear_left_wheel_joint</joint_name>
-      <joint_name>rear_right_wheel_joint</joint_name>
-    </plugin>
-    <plugin filename="gz_ros2_control-system" name="gz_ros2_control::GazeboSimROS2ControlPlugin">
-      <parameters>$(find gazebo_ackermann_steering_vehicle)/config/gz_ros2_control.yaml</parameters>
-    </plugin>
-  </gazebo>
 </robot>
