Commit message: fix: fixed tf transform front wheels joints

File: src/platform_description/urdf/gazebo_ros2_control.xacro (robot description, xacro)
@@ -5,4 +5,14 @@
       <plugin>gz_ros2_control/GazeboSimSystem</plugin>
     </hardware>
+      <joint name="front_left_wheel_joint">
+        <state_interface name="position"/>
+        <state_interface name="velocity"/>
+        <state_interface name="effort"/>
+      </joint>
+      <joint name="front_right_wheel_joint">
+        <state_interface name="position"/>
+        <state_interface name="velocity"/>
+        <state_interface name="effort"/>
+      </joint>
     <joint name="front_left_steering_joint">
       <command_interface name="position">

Commit message: fix: resolve missing odom TF and joint state conflicts - Remapped 'tf_odometry' to 'tf' in Gazebo plugin for correct odom -> base_footprint tree. - Disabled Gazebo 'joint_states' bridge to prevent conflicts with ROS joint_state_broadcaster. - Added passive front wheels as state-only interfaces in ros2_control URDF. - Fixed config file paths in the main launch file.

File: src/platform_description/urdf/gazebo_ros2_control.xacro (robot description, xacro)
@@ -41,4 +41,14 @@
       <state_interface name="effort"/>
     </joint>
+        <joint name="front_left_wheel_joint">
+      <state_interface name="position"/>
+      <state_interface name="velocity"/>
+      <state_interface name="effort"/>
+    </joint>
+    <joint name="front_right_wheel_joint">
+      <state_interface name="position"/>
+      <state_interface name="velocity"/>
+      <state_interface name="effort"/>
+    </joint>
   </ros2_control>
   <gazebo>
@@ -54,4 +64,7 @@
     <plugin filename="gz_ros2_control-system" name="gz_ros2_control::GazeboSimROS2ControlPlugin">
       <parameters>$(find platform_bringup)/config/gz_ros2_control.yaml</parameters>
+      <ros>
+        <remapping>/ackermann_steering_controller/tf_odometry:=/tf</remapping>
+      </ros>
     </plugin>
   </gazebo>
