Commit message: feat: add depth camera and xacro variables for camera

File: src/platform_description/urdf/common_properties.xacro (robot description, xacro)
@@ -11,3 +11,5 @@
     <xacro:property name="max_wheel_angular_velocity" value="100.0"/>
     <xacro:property name="max_effort" value="30.0" />
+    <xacro:property name="base_length" value="0.23"/>
+    <xacro:property name="base_height" value="0.10"/>
 </robot>

Commit message: refactor(urdf): move hardcoded link dimensions and inertias to xacro properties

File: src/platform_description/urdf/common_properties.xacro (robot description, xacro)
@@ -11,3 +11,14 @@
     <xacro:property name="max_wheel_angular_velocity" value="100.0"/>
     <xacro:property name="max_effort" value="30.0" />
+<!-- Platform properties -->
+    <xacro:property name="platform_mass" value="1.5"/>
+    <xacro:property name="platform_length" value="0.22"/>
+    <xacro:property name="platform_width" value="0.23"/>
+    <xacro:property name="platform_height" value="0.03"/>
+    <xacro:property name="platform_offset_x" value="-0.0075"/>
+    <xacro:property name="platform_offset_y" value="0.0"/>
+    <xacro:property name="platform_offset_z" value="0.0001"/>
+<!-- Wheel bar properties -->
+    <xacro:property name="wheel_bar_mass" value="0.05"/>
+    <xacro:property name="wheel_bar_radius" value="0.01"/>
 </robot>

File: src/platform_description/urdf/platform_base.xacro (robot description, xacro)
@@ -29,16 +29,16 @@
   <link name="platform_link">
       <visual>
-          <geometry> <box size="0.22 0.23 0.03"/> </geometry>
+          <geometry> <box size="${platform_length} ${platform_width} ${platform_height}"/> </geometry>
           <material name="red"/>
       </visual>
       <collision>
-          <geometry> <box size="0.22 0.23 0.03"/> </geometry>
+          <geometry> <box size="${platform_length} ${platform_width} ${platform_height}"/> </geometry>
       </collision>
-      <xacro:box_inertia m="1.5" l="0.22" w="0.23" h="0.03" xyz="0 0 0" rpy="0 0 0"/>
+      <xacro:box_inertia m="${platform_mass}" l="${platform_length}" w="${platform_width}" h="${platform_height}" xyz="0 0 0" rpy="0 0 0"/>
   </link>
   <joint name="base_platform_joint" type="fixed">
       <parent link="base_link"/>
       <child link="platform_link"/>
-      <origin xyz="-0.0075 0 0.0001" rpy="0 0 0"/>
+      <origin xyz="${platform_offset_x} ${platform_offset_y} ${platform_offset_z}" rpy="0 0 0"/>
   </joint>
 <!-- ============================================== -->
@@ -48,8 +48,8 @@
       <link name="${prefix}_wheel_bar">
           <visual>
-              <geometry> <cylinder radius="0.01" length="${length}"/> </geometry>
+              <geometry> <cylinder radius="${wheel_bar_radius}" length="${length}"/> </geometry>
               <origin xyz="0.0 0.0 0.0" rpy="-1.57 0.0 0.0"/>
           </visual>
-          <xacro:cylinder_inertia m="0.05" r="0.01" h="${length}" xyz="0 0 0" rpy="-1.57 0 0"/>
+          <xacro:cylinder_inertia m="${wheel_bar_mass}" r="${wheel_bar_radius}" h="${length}" xyz="0 0 0" rpy="-1.57 0 0"/>
       </link>
       <joint name="base_${prefix}_wheel_bar" type="fixed">

Commit message: refactor: changed to parameters in depth_camera from base_ to chassis_

File: src/platform_description/urdf/common_properties.xacro (robot description, xacro)
@@ -11,5 +11,3 @@
     <xacro:property name="max_wheel_angular_velocity" value="100.0"/>
     <xacro:property name="max_effort" value="30.0" />
-    <xacro:property name="base_length" value="0.23"/>
-    <xacro:property name="base_height" value="0.10"/>
 </robot>

File: src/platform_description/urdf/depth_camera.xacro (robot description, xacro)
@@ -24,5 +24,5 @@
         <parent link="base_link"/>
         <child link="depth_camera_link"/>
-        <origin xyz="${(base_length + camera_length) / 2.0} 0 ${base_height / 2.0}" rpy="0 0 0" />
+        <origin xyz="${(chassis_length + camera_length) / 2.0} 0 ${chassis_height / 2.0}" rpy="0 0 0" />
     </joint>
     <joint name="depth_camera_optical_joint" type="fixed">
