Commit message: refactor: changed to parameters in camera from base_ to chassis_

File: src/platform_description/urdf/camera.xacro (robot description, xacro)
@@ -22,5 +22,5 @@
         <parent link="base_link" />
         <child link="camera_link" />
-        <origin xyz="${(base_length + camera_length) / 2.0} 0 ${base_height / 2.0}" rpy="0 0 0" />
+        <origin xyz="${(chassis_length + camera_length) / 2.0} 0 ${chassis_height / 2.0}" rpy="0 0 0" />
     </joint>
     <link name="camera_link_optical" />

Commit message: refactor: changed parameters of position for the cameras

File: src/platform_description/urdf/camera.xacro (robot description, xacro)
@@ -22,5 +22,5 @@
         <parent link="base_link" />
         <child link="camera_link" />
-        <origin xyz="${(chassis_length + camera_length) / 2.0} 0 ${chassis_height / 2.0}" rpy="0 0 0" />
+        <origin xyz="${-(chassis_length + camera_length) / 4.0} 0 ${chassis_height + camera_height}" rpy="0 0 0" />
     </joint>
     <link name="camera_link_optical" />

File: src/platform_description/urdf/depth_camera.xacro (robot description, xacro)
@@ -24,5 +24,5 @@
         <parent link="base_link"/>
         <child link="depth_camera_link"/>
-        <origin xyz="${(chassis_length + camera_length) / 2.0} 0 ${chassis_height / 2.0}" rpy="0 0 0" />
+        <origin xyz="${-(chassis_length + camera_length) / 3.0} 0 ${chassis_height + camera_height}" rpy="0 0 0" />
     </joint>
     <joint name="depth_camera_optical_joint" type="fixed">

Commit message: change to default camera

File: src/platform_description/urdf/camera.xacro (robot description, xacro)
@@ -1,59 +1,58 @@
 <?xml version="1.0"?>
 <robot xmlns:xacro="http://www.ros.org/wiki/xacro">
-    <xacro:property name="camera_length" value="0.01" />
-    <xacro:property name="camera_width" value="0.15" />
-    <xacro:property name="camera_height" value="0.05" />
-    <link name="camera_link">
-        <visual>
-            <geometry>
-                <box size="${camera_length} ${camera_width} ${camera_height}" />
-            </geometry>
-            <material name="xd" />
-        </visual>
-        <collision>
-            <geometry>
-                <box size="${camera_length} ${camera_width} ${camera_height}" />
-            </geometry>
-        </collision>
-        <xacro:box_inertia m="0.1" x="${camera_length}" y="${camera_width}" z="${camera_height}"
-                           o_xyz="0 0 0" o_rpy="0 0 0" />
-    </link>
-    <joint name="base_camera_joint" type="fixed">
-        <parent link="base_link" />
-        <child link="camera_link" />
-        <origin xyz="${-(chassis_length + camera_length) / 4.0} 0 ${chassis_height + camera_height}" rpy="0 0 0" />
-    </joint>
-    <link name="camera_link_optical" />
-    <joint name="camera_optical_joint" type="fixed">
-        <origin xyz="0 0 0" rpy="${-pi/2} 0 ${-pi/2}"/>
-        <parent link="camera_link"/>
-        <child link="camera_link_optical"/>
-    </joint>
-    <gazebo reference="camera_link">
-        <sensor name="camera" type="camera">
-            <camera>
-                <horizontal_fov>1.3962634</horizontal_fov>
-                <image>
-                    <width>640</width>
-                    <height>480</height>
-                    <format>R8G8B8</format>
-                </image>
-                <clip>
-                    <near>0.1</near>
-                    <far>15</far>
-                </clip>
-                <noise>
-                    <type>gaussian</type>
-                    <mean>0.0</mean>
-                    <stddev>0.007</stddev>
-                </noise>
-                <optical_frame_id>camera_link_optical</optical_frame_id>
-                <camera_info_topic>camera/camera_info</camera_info_topic>
-            </camera>
-            <always_on>1</always_on>
-            <update_rate>20</update_rate>
-            <visualize>true</visualize>
-            <topic>camera/image_raw</topic>
-        </sensor>
-    </gazebo>
+  <xacro:property name="camera_length" value="0.01" />
+  <xacro:property name="camera_width"  value="0.15" />
+  <xacro:property name="camera_height" value="0.05" />
+  <link name="camera_link">
+    <visual>
+      <geometry>
+        <box size="${camera_length} ${camera_width} ${camera_height}" />
+      </geometry>
+      <material name="black" />
+    </visual>
+    <collision>
+      <geometry>
+        <box size="${camera_length} ${camera_width} ${camera_height}" />
+      </geometry>
+    </collision>
+    <xacro:box_inertia m="0.1" l="${camera_length}" w="${camera_width}" h="${camera_height}"
+                       xyz="0 0 0" rpy="0 0 0" />
+  </link>
+  <joint name="base_camera_joint" type="fixed">
+    <parent link="base_link" />
+    <child link="camera_link" />
+    <origin xyz="${-(chassis_length + camera_length) / 4.0} 0 ${chassis_height + camera_height}" rpy="0 0 0" />
+  </joint>
+  <link name="camera_link_optical" />
+  <joint name="camera_optical_joint" type="fixed">
+    <origin xyz="0 0 0" rpy="${-pi/2} 0 ${-pi/2}"/>
+    <parent link="camera_link"/>
+    <child link="camera_link_optical"/>
+  </joint>
+ <gazebo reference="camera_link">
+    <sensor name="camera_sensor" type="camera">
+      <topic>camera/image_raw</topic>
+      <update_rate>20</update_rate>
+      <always_on>1</always_on>
+      <visualize>true</visualize>
+      <gz_frame_id>camera_link_optical</gz_frame_id>
+      <camera>
+        <horizontal_fov>1.3962634</horizontal_fov>
+        <image>
+          <width>640</width>
+          <height>480</height>
+          <format>R8G8B8</format>
+        </image>
+        <clip>
+          <near>0.1</near>
+          <far>15</far>
+        </clip>
+        <noise>
+          <type>gaussian</type>
+          <mean>0.0</mean>
+          <stddev>0.007</stddev>
+        </noise>
+      </camera>
+    </sensor>
+  </gazebo>
 </robot>

File: src/platform_description/urdf/gazebo_ros2_control.xacro (robot description, xacro)
@@ -5,4 +5,5 @@
       <plugin>gz_ros2_control/GazeboSimSystem</plugin>
     </hardware>
+      <!-- Przednie kola: stany-->
       <joint name="front_left_wheel_joint">
         <state_interface name="position"/>
@@ -15,4 +16,5 @@
         <state_interface name="effort"/>
       </joint>
+    <!-- Zwrotnice: komenda pozycji -->
     <joint name="front_left_steering_joint">
       <command_interface name="position">
@@ -33,4 +35,5 @@
       <state_interface name="effort"/>
     </joint>
+    <!-- Naped tylny: komenda predkosci -->
     <joint name="rear_left_wheel_joint">
       <command_interface name="velocity">
@@ -51,31 +54,10 @@
       <state_interface name="effort"/>
     </joint>
-        <joint name="front_left_wheel_joint">
-      <state_interface name="position"/>
-      <state_interface name="velocity"/>
-      <state_interface name="effort"/>
-    </joint>
-    <joint name="front_right_wheel_joint">
-      <state_interface name="position"/>
-      <state_interface name="velocity"/>
-      <state_interface name="effort"/>
-    </joint>
   </ros2_control>
-  <gazebo>
-    <plugin filename="gz-sim-joint-state-publisher-system" name="gz::sim::systems::JointStatePublisher">
-      <topic>joint_states</topic>
-      <joint_name>front_left_steering_joint</joint_name>
-      <joint_name>front_right_steering_joint</joint_name>
-      <joint_name>front_left_wheel_joint</joint_name>
-      <joint_name>front_right_wheel_joint</joint_name>
-      <joint_name>rear_left_wheel_joint</joint_name>
-      <joint_name>rear_right_wheel_joint</joint_name>
-    </plugin>
-    <plugin filename="gz_ros2_control-system" name="gz_ros2_control::GazeboSimROS2ControlPlugin">
-      <parameters>$(find platform_bringup)/config/gz_ros2_control.yaml</parameters>
-      <ros>
-        <remapping>/ackermann_steering_controller/tf_odometry:=/tf</remapping>
-      </ros>
-    </plugin>
-  </gazebo>
+<gazebo>
+  <plugin filename="gz_ros2_control-system"
+          name="gz_ros2_control::GazeboSimROS2ControlPlugin">
+    <parameters>$(find platform_bringup)/config/gz_ros2_control.yaml</parameters>
+  </plugin>
+</gazebo>
 </robot>

File: src/platform_description/urdf/platform.urdf.xacro (robot description, xacro)
@@ -4,5 +4,6 @@
     <xacro:include filename="inertials.xacro"/>
     <xacro:include filename="platform_base.xacro"/>
-    <xacro:include filename="depth_camera.xacro"/>
+    <xacro:include filename="camera.xacro"/>
+    <!-- <xacro:include filename="depth_camera.xacro"/> -->
     <xacro:include filename="lidar.xacro"/>
     <xacro:include filename="gazebo_ros2_control.xacro"/>
